Commit message: fixed things

File: src/robotics_model_3dof/robot/visual/TeeTyBot.xacro (robot description, xacro)
@@ -1,71 +1,79 @@
 <?xml version="1.0"?>
 <robot xmlns:xacro="http://www.ros.org/wiki/xacro" name="example">
-    <link name="link_0">
-        <visual>
-            <origin rpy="0 0 0" xyz="0.0 0.0 0.0" />
-            <geometry>
-                <mesh filename="file:///$(find robotics_model_3dof)/meshes/link_0.stl" />
-            </geometry>
-        </visual>
-    </link>
-    <link name="link_1">
-        <visual>
-            <origin rpy="0 0 0" xyz="0.0 0.0 0.0" />
-            <geometry>
-                <mesh filename="file:///$(find robotics_model_3dof)/meshes/link_1.stl" />
-            </geometry>
-        </visual>
-    </link>
-    <joint name="joint_1" type="revolute">
-        <origin xyz="0.0 0.0 0.2" rpy="0.0 0.0 0.0"/>
-        <parent link="link_0"/>
-        <child link="link_1"/>
-        <axis xyz="0.0 0.0 1.0"/>
-        <limit lower="0" upper="6.28" effort="100.0" velocity="100.0"/>
-    </joint>
-    <link name="link_2">
-        <visual>
-            <origin rpy="3.14 0 0" xyz="0.0 0.0 0.0" />
-            <geometry>
-                <mesh filename="file:///$(find robotics_model_3dof)/meshes/link_2.stl" />
-            </geometry>
-        </visual>
-    </link>
-    <joint name="joint_2" type="revolute">
-        <origin xyz="0.0 -0.12 0.0" rpy="1.5708 0 0"/>
-        <parent link="link_1"/>
-        <child link="link_2"/>
-        <axis xyz="0.0 0.0 1.0"/>
-        <limit lower="0" upper="3.14" effort="100.0" velocity="100.0"/>
-    </joint>
-    <link name="link_3">
-        <visual>
-            <origin rpy="3.14 0 0" xyz="0.0 0.0 0.0" />
-            <geometry>
-                <mesh filename="file:///$(find robotics_model_3dof)/meshes/link_3.stl" />
-            </geometry>
-        </visual>
-    </link>
-    <joint name="joint_3" type="revolute">
-        <origin xyz="0.25 0.0 -0.1" rpy="0.0 0.0 0.0"/>
-        <parent link="link_2"/>
-        <child link="link_3"/>
-        <axis xyz="0.0 0.0 1.0"/>
-        <limit lower="0" upper="3.14" effort="100.0" velocity="100.0"/>
-    </joint>
-    <link name="end_effector">
-        <visual>
-            <origin rpy="0 1.57 0" xyz="0.0 0.0 0.0" />
-            <geometry>
-                <mesh filename="file:///$(find robotics_model_3dof)/meshes/end_effector.stl" />
-            </geometry>
-        </visual>
-    </link>
-    <joint name="joint_4" type="fixed">
-        <origin xyz="0.28 0.0 0.0" rpy="0.0 0.0 0.0"/>
-        <parent link="link_3"/>
-        <child link="end_effector"/>
-        <axis xyz="0.0 0.0 0.0"/>
-        <limit lower="0.0" upper="6.28" effort="100.0" velocity="100.0"/>
-    </joint>
+  <link name="link_0">
+    <visual>
+      <geometry>
+        <mesh filename="file:///$(find robotics_model_3dof)/meshes/link_0.stl"/>
+      </geometry>
+    </visual>
+  </link>
+  <link name="link_1">
+    <visual>
+      <geometry>
+        <mesh filename="file:///$(find robotics_model_3dof)/meshes/link_1.stl"/>
+      </geometry>
+    </visual>
+  </link>
+  <joint name="joint_1" type="revolute">
+    <parent link="link_0"/>
+    <child link="link_1"/>
+    <origin xyz="0 0 0.2" rpy="0 0 0"/>
+    <axis xyz="0 0 1"/>
+    <limit
+      lower="-3.1459"
+      upper="3.1459"
+      velocity="1000.0"
+      effort="1000.0"/>
+  </joint>
+  <link name="link_2">
+    <visual>
+      <origin xyz="0.0 0.0 0.0" rpy="0 0 ${-3.14/2}"/>
+      <geometry>
+        <mesh filename="file:///$(find robotics_model_3dof)/meshes/link_2.stl"/>
+      </geometry>
+    </visual>
+  </link>
+  <joint name="joint_2" type="revolute">
+    <parent link="link_1"/>
+    <child link="link_2"/>
+    <origin xyz="0.0 -0.12 0.0" rpy="${-3.14/2} 0 0"/>
+    <axis xyz="0 0 1"/>
+    <limit
+      lower="-3.1459"
+      upper="3.1459"
+      velocity="1000.0"
+      effort="1000.0"/>
+  </joint>
+  <link name="link_3">
+    <visual>
+      <origin xyz="0.0 0.0 0.0" rpy="0 0 ${-3.14/2}"/>
+      <geometry>
+        <mesh filename="file:///$(find robotics_model_3dof)/meshes/link_3.stl"/>
+      </geometry>
+    </visual>
+  </link>
+  <joint name="joint_3" type="revolute">
+    <parent link="link_2"/>
+    <child link="link_3"/>
+    <origin xyz="0.0 -0.25 0.1" rpy="0 0 0"/>
+    <axis xyz="0 0 1"/>
+    <limit
+      lower="-3.1459"
+      upper="3.1459"
+      velocity="1000.0"
+      effort="1000.0"/>
+  </joint>
+  <link name="end_effector">
+    <visual>
+      <origin xyz="0.0 0.0 0.0" rpy="0 0 0"/>
+      <geometry>
+        <mesh filename="file:///$(find robotics_model_3dof)/meshes/end_effector.stl"/>
+      </geometry>
+    </visual>
+  </link>
+  <joint name="joint_end_effector" type="fixed">
+    <parent link="link_3"/>
+    <child link="end_effector"/>
+    <origin xyz="0.0 -0.28 0.0" rpy="${3.14/2} 0 0"/>
+  </joint>
 </robot>

File: src/robotics_model_3dof/robot/visual/my-robot.xacro (robot description, xacro)
@@ -1,79 +1,71 @@
 <?xml version="1.0"?>
 <robot xmlns:xacro="http://www.ros.org/wiki/xacro" name="example">
-  <link name="link_0">
-    <visual>
-      <geometry>
-        <mesh filename="file:///$(find example_description)/meshes/link_0.stl"/>
-      </geometry>
-    </visual>
-  </link>
-  <link name="link_1">
-    <visual>
-      <geometry>
-        <mesh filename="file:///$(find example_description)/meshes/link_1.stl"/>
-      </geometry>
-    </visual>
-  </link>
-  <joint name="joint_1" type="revolute">
-    <parent link="link_0"/>
-    <child link="link_1"/>
-    <origin xyz="0 0 0.2" rpy="0 0 0"/>
-    <axis xyz="0 0 1"/>
-    <limit
-      lower="-3.1459"
-      upper="3.1459"
-      velocity="1000.0"
-      effort="1000.0"/>
-  </joint>
-  <link name="link_2">
-    <visual>
-      <origin xyz="0.0 0.0 0.0" rpy="0 0 ${-3.14/2}"/>
-      <geometry>
-        <mesh filename="file:///$(find example_description)/meshes/link_2.stl"/>
-      </geometry>
-    </visual>
-  </link>
-  <joint name="joint_2" type="revolute">
-    <parent link="link_1"/>
-    <child link="link_2"/>
-    <origin xyz="0.0 -0.12 0.0" rpy="${-3.14/2} 0 0"/>
-    <axis xyz="0 0 1"/>
-    <limit
-      lower="-3.1459"
-      upper="3.1459"
-      velocity="1000.0"
-      effort="1000.0"/>
-  </joint>
-  <link name="link_3">
-    <visual>
-      <origin xyz="0.0 0.0 0.0" rpy="0 0 ${-3.14/2}"/>
-      <geometry>
-        <mesh filename="file:///$(find example_description)/meshes/link_3.stl"/>
-      </geometry>
-    </visual>
-  </link>
-  <joint name="joint_3" type="revolute">
-    <parent link="link_2"/>
-    <child link="link_3"/>
-    <origin xyz="0.0 -0.25 0.1" rpy="0 0 0"/>
-    <axis xyz="0 0 1"/>
-    <limit
-      lower="-3.1459"
-      upper="3.1459"
-      velocity="1000.0"
-      effort="1000.0"/>
-  </joint>
-  <link name="end_effector">
-    <visual>
-      <origin xyz="0.0 0.0 0.0" rpy="0 0 0"/>
-      <geometry>
-        <mesh filename="file:///$(find example_description)/meshes/end_effector.stl"/>
-      </geometry>
-    </visual>
-  </link>
-  <joint name="joint_end_effector" type="fixed">
-    <parent link="link_3"/>
-    <child link="end_effector"/>
-    <origin xyz="0.0 -0.28 0.0" rpy="${3.14/2} 0 0"/>
-  </joint>
+    <link name="link_0">
+        <visual>
+            <origin rpy="0 0 0" xyz="0.0 0.0 0.0" />
+            <geometry>
+                <mesh filename="file:///$(find robotics_model_3dof)/meshes/link_0.stl" />
+            </geometry>
+        </visual>
+    </link>
+    <link name="link_1">
+        <visual>
+            <origin rpy="0 0 0" xyz="0.0 0.0 0.0" />
+            <geometry>
+                <mesh filename="file:///$(find robotics_model_3dof)/meshes/link_1.stl" />
+            </geometry>
+        </visual>
+    </link>
+    <joint name="joint_1" type="revolute">
+        <origin xyz="0.0 0.0 0.2" rpy="0.0 0.0 0.0"/>
+        <parent link="link_0"/>
+        <child link="link_1"/>
+        <axis xyz="0.0 0.0 1.0"/>
+        <limit lower="0" upper="6.28" effort="100.0" velocity="100.0"/>
+    </joint>
+    <link name="link_2">
+        <visual>
+            <origin rpy="3.14 0 0" xyz="0.0 0.0 0.0" />
+            <geometry>
+                <mesh filename="file:///$(find robotics_model_3dof)/meshes/link_2.stl" />
+            </geometry>
+        </visual>
+    </link>
+    <joint name="joint_2" type="revolute">
+        <origin xyz="0.0 -0.12 0.0" rpy="1.5708 0 0"/>
+        <parent link="link_1"/>
+        <child link="link_2"/>
+        <axis xyz="0.0 0.0 1.0"/>
+        <limit lower="0" upper="3.14" effort="100.0" velocity="100.0"/>
+    </joint>
+    <link name="link_3">
+        <visual>
+            <origin rpy="3.14 0 0" xyz="0.0 0.0 0.0" />
+            <geometry>
+                <mesh filename="file:///$(find robotics_model_3dof)/meshes/link_3.stl" />
+            </geometry>
+        </visual>
+    </link>
+    <joint name="joint_3" type="revolute">
+        <origin xyz="0.25 0.0 -0.1" rpy="0.0 0.0 0.0"/>
+        <parent link="link_2"/>
+        <child link="link_3"/>
+        <axis xyz="0.0 0.0 1.0"/>
+        <limit lower="0" upper="3.14" effort="100.0" velocity="100.0"/>
+    </joint>
+    <link name="end_effector">
+        <visual>
+            <origin rpy="0 1.57 0" xyz="0.0 0.0 0.0" />
+            <geometry>
+                <mesh filename="file:///$(find robotics_model_3dof)/meshes/end_effector.stl" />
+            </geometry>
+        </visual>
+    </link>
+    <joint name="joint_4" type="fixed">
+        <origin xyz="0.28 0.0 0.0" rpy="0.0 0.0 0.0"/>
+        <parent link="link_3"/>
+        <child link="end_effector"/>
+        <axis xyz="0.0 0.0 0.0"/>
+        <limit lower="0.0" upper="6.28" effort="100.0" velocity="100.0"/>
+    </joint>
 </robot>
